File: A3660/A3660.sch (EAGLE design)
At the start: 2 parts, among them CN100 KEL8817-200-170S-F, U102 MC68040/68060

Commit message: Added and changed some in library. Added schematics for CPU, Cpuclockdriver and some of the latches
Parts:
- added C100A: 10nF, A3660:C0805
- added C101A, C103A, C105A: 100nF, A3660:C0805
- added C101B, C214A, C214A5, C214A6, C214A7, C214A8, C214A9, C215A, C216A, C217A: 330nF, A3660:C0805
- added C102A, C102D: 220nF, A3660:C0805
- added C102B, C102E: 22uF, A3660:SMD-ELECTROLYTE
- added C102C, C102F: 220pF, A3660:C0805
- added C501: 10uF, A3660:C0805
- added FB100: (no value), A3660:FERRITE
- added R100, R103: 1, A3660:R0805
- added R101A, R101B, R102: 22, A3660:R0805
- added R104, R105: 4.7K, A3660:R0805
- added R107, R108: 33, A3660:R0805
- added RP100A, RP100B, RP402A, RP403A, RP403B, RP404A, RP404B, RP405A, RP405B, RP405C: 1K, A3660:RP743-8
- added RP101, RP102, RP103, RP104, RP105, RP106, RP107, RP108: 22, A3660:RP743-8
- added RP400A, RP400B: (no value), A3660:RP743-8
- added U$1: 2X22-2MM, adafruit:2X22-2MM
- added U$10, U$11, U$7, U$8, U$9, U214, U215, U216, U217: 74FCT543A, A3660:74FCT543A
- added U100: OSCILLATOR, A3660:OSCILLATOR
- added U101: 74F1803, A3660:74F1803
- added U103: DELAYLINE, A3660:DELAYLINE
- added U105: 74F04, A3660:74F04
- added VR1: LT1084-3.3, A3660:LT1084-3.3
Connections:
- new net +3V3: C102A.1, C102B.1, C102C.1, C102D.1, C102E.1, C102F.1, C501.1, U102.VCC0, U102.VCC1, U102.VCC10, U102.VCC11, U102.VCC12, U102.VCC13, U102.VCC14, U102.VCC15, U102.VCC16, U102.VCC17, U102.VCC18, U102.VCC19, U102.VCC2, U102.VCC20, U102.VCC21, U102.VCC22, U102.VCC23, U102.VCC24, U102.VCC25, U102.VCC26, U102.VCC27, U102.VCC28, U102.VCC29, U102.VCC3, U102.VCC30, U102.VCC31, U102.VCC32, U102.VCC33, U102.VCC34, U102.VCC35, U102.VCC36, U102.VCC37, U102.VCC38, U102.VCC39, U102.VCC4, U102.VCC40, U102.VCC5, U102.VCC6, U102.VCC7, U102.VCC8, U102.VCC9, VR1.OUT
- new net +5V: C101A.1, C101B.1, C105A.2, C214A.2, C214A5.2, C214A6.2, C214A7.2, C214A8.2, C214A9.2, C215A.2, C216A.2, C217A.2, CN100.+5V-0, CN100.+5V-1, CN100.+5V-10, CN100.+5V-11, CN100.+5V-12, CN100.+5V-13, CN100.+5V-14, CN100.+5V-15, CN100.+5V-16, CN100.+5V-17, CN100.+5V-18, CN100.+5V-19, CN100.+5V-2, CN100.+5V-20, CN100.+5V-21, CN100.+5V-22, CN100.+5V-23, CN100.+5V-3, CN100.+5V-4, CN100.+5V-5, CN100.+5V-6, CN100.+5V-7, CN100.+5V-8, CN100.+5V-9, R104.1, RP400B.1, RP400B.2, RP400B.3, RP400B.4, RP402A.1, RP402A.2, RP402A.3, RP402A.4, RP403A.1, RP403A.2, RP403A.3, RP403A.4, RP403B.1, RP403B.2, RP403B.3, RP403B.4, RP404A.1, RP404A.2, RP404A.3, RP404A.4, RP404B.1, RP404B.2, RP404B.3, RP404B.4, RP405A.1, RP405A.2, RP405A.3, RP405A.4, RP405B.1, RP405B.2, RP405B.3, RP405B.4, RP405C.1, RP405C.2, RP405C.3, RP405C.4, U$10.VCC, U$11.VCC, U$7.VCC, U$8.VCC, U$9.VCC, U101.VCC, U105.VCC, U214.VCC, U215.VCC, U216.VCC, U217.VCC, VR1.IN
- new net 10NS: R101A.2, U103.TAP2
- new net 5NS: R101B.2, U103.TAP1
- new net A0: CN100.A0, RP108.4, RP400A.5
- new net A1: CN100.A1, RP108.3, RP400A.6
- new net A10: CN100.A10, RP106.2
- new net A11: CN100.A11, RP106.1
- new net A12: CN100.A12, RP105.4
- new net A13: CN100.A13, RP105.3
- new net A14: CN100.A14, RP105.2
- new net A15: CN100.A15, RP105.1
- new net A16: CN100.A16, RP104.4
- new net A17: CN100.A17, RP104.3
- new net A18: CN100.A18, RP104.2
- new net A19: CN100.A19, RP104.1
- new net A2: CN100.A2, RP108.2, RP400A.7
- new net A20: CN100.A20, RP103.4
- new net A21: CN100.A21, RP103.3
- new net A22: CN100.A22, RP103.2
- new net A23: CN100.A23, RP103.1
- new net A24: CN100.A24, RP102.4
- new net A25: CN100.A25, RP102.3
- new net A26: CN100.A26, RP102.2
- new net A27: CN100.A27, RP102.1
- new net A28: CN100.A28, RP101.4
- new net A29: CN100.A29, RP101.3
- new net A3: CN100.A3, RP108.1, RP400A.8
- new net A30: CN100.A30, RP101.2
- new net A31: CN100.A31, RP101.1
- new net A4: CN100.A4, RP107.4
- new net A5: CN100.A5, RP107.3
- new net A6: CN100.A6, RP107.2
- new net A7: CN100.A7, RP107.1
- new net A8: CN100.A8, RP106.4
- new net A9: CN100.A9, RP106.3
- new net CLK90: CN100.EXT90, R101A.1
- new net CPUCLK: CN100.EXTCPU, R102.2
- new net D0: CN100.D0
- new net D1: CN100.D1
- new net D10: CN100.D10
- new net D11: CN100.D11
- new net D12: CN100.D12
- new net D13: CN100.D13
- new net D14: CN100.D14
- new net D15: CN100.D15
- new net D16: CN100.D16, U216.B0
- new net D17: CN100.D17, U216.B1
- new net D18: CN100.D18, U216.B2
- new net D19: CN100.D19, U216.B3
- new net D2: CN100.D2
- new net D20: CN100.D20, U216.B4
- new net D21: CN100.D21, U216.B5
- new net D22: CN100.D22, U216.B6
- new net D23: CN100.D23, U216.B7
- new net D24: CN100.D24, U214.B0, U215.B0, U217.B0
- new net D25: CN100.D25, U214.B1, U215.B1, U217.B1
- new net D26: CN100.D26, U214.B2, U215.B2, U217.B2
- new net D27: CN100.D27, U214.B3, U215.B3, U217.B3
- new net D28: CN100.D28, U214.B4, U215.B4, U217.B4
- new net D29: CN100.D29, U214.B5, U215.B5, U217.B5
- new net D3: CN100.D3
- new net D30: CN100.D30, U214.B6, U215.B6, U217.B6
- new net D31: CN100.D31, U214.B7, U215.B7, U217.B7
- new net D4: CN100.D4
- new net D5: CN100.D5
- new net D6: CN100.D6
- new net D7: CN100.D7
- new net D8: CN100.D8
- new net D9: CN100.D9
- new net LEBUS0: U214.!LEBA
- new net LEBUS1: U215.!LEBA
- new net LEBUS2: U216.!LEBA
- new net LEBUS3: U217.!LEBA
- new net N$10: RP100B.8
- new net N$11: U101.D2, U101.D3, U105.1!Y
- new net N$12: R103.1, U101.D0, U101.D1, U101.O0, U101.O1, U105.1A
- new net N$13: R102.1, U101.O2
- new net N$14: U101.O3, U103.IN
- new net N$15: C103A.1, U103.VCC
- new net N$16: U101.GND
- new net N$17: R101B.1
- new net N$18: U102.R_W, U105.2A
- new net N$19: RP400A.3
- new net N$2: R107.1, U102.SIZ1
- new net N$20: RP400A.2
- new net N$21: RP400A.1
- new net N$23: RP400B.8
- new net N$3: R108.1, U102.SIZ0
- new net N$4: FB100.1, U102._TS
- new net N$47: U$7.!CEBA
- new net N$48: U$7.!OEAB
- new net N$49: U$7.!OEBA
- new net N$5: C100A.1, U100.VCC
- new net N$50: U$7.!LEBA
- new net N$51: U$7.!LEAB
- new net N$52: U$7.!CEAB
- new net N$53: U$8.!CEBA
- new net N$54: U$8.!OEAB
- new net N$55: U$8.!OEBA
- new net N$56: U$8.!LEBA
- new net N$57: U$8.!LEAB
- new net N$58: U$8.!CEAB
- new net N$59: U$9.!CEBA
- new net N$6: R100.1, U100.OUT
- new net N$60: U$9.!OEAB
- new net N$61: U$9.!OEBA
- new net N$62: U$9.!LEBA
- new net N$63: U$9.!LEAB
- new net N$64: U$9.!CEAB
- new net N$65: U$10.!CEBA
- new net N$66: U$10.!OEAB
- new net N$67: U$10.!OEBA
- new net N$68: U$10.!LEBA
- new net N$69: U$10.!LEAB
- new net N$7: RP400A.4
- new net N$70: U$10.!CEAB
- new net N$71: U$11.!CEBA
- new net N$72: U$11.!OEAB
- new net N$73: U$11.!OEBA
- new net N$74: U$11.!LEBA
- new net N$75: U$11.!LEAB
- new net N$76: U$11.!CEAB
- new net N$8: RP100B.6
- new net N$9: RP100B.7
- new net OEBUS0: U214.!OEAB, U214.!OEBA
- new net OEBUS1: U215.!OEAB, U215.!OEBA
- new net OEBUS2: U216.!OEAB, U216.!OEBA
- new net OEBUS3: U217.!OEAB, U217.!OEBA
- new net R_W060: RP400B.7, U214.!CEAB, U215.!CEAB, U216.!CEAB, U217.!CEAB
- new net TCK: RP100B.5, U102.TCK
- new net TDI: RP100A.7, U102.TDI
- new net TMS: RP100A.8, U102.TMS
- new net _060EMUL: R105.1, U102._CDIS, U102._MDIS
- new net _R_W060: U105.2!Y, U214.!CEBA, U215.!CEBA, U216.!CEBA, U217.!CEBA
- new net _TBI: RP100A.5, U102._TBI
- new net _TRST: RP100A.6, U102._TRST
- new net _TS: FB100.2, R104.2
- net 060A0: now also RP108.5
- net 060A1: now also RP108.6
- net 060A10: now also RP106.7
- net 060A11: now also RP106.8
- net 060A12: now also RP105.5
- net 060A13: now also RP105.6
- net 060A14: now also RP105.7
- net 060A15: now also RP105.8
- net 060A16: now also RP104.5
- net 060A17: now also RP104.6
- net 060A18: now also RP104.7
- net 060A19: now also RP104.8
- net 060A2: now also RP108.7
- net 060A20: now also RP103.5
- net 060A21: now also RP103.6
- net 060A22: now also RP103.7
- net 060A23: now also RP103.8
- net 060A24: now also RP102.5
- net 060A25: now also RP102.6
- net 060A26: now also RP102.7
- net 060A27: now also RP102.8
- net 060A28: now also RP101.5
- net 060A29: now also RP101.6
- net 060A3: now also RP108.8
- net 060A30: now also RP101.7
- net 060A31: now also RP101.8
- net 060A4: now also RP107.5
- net 060A5: now also RP107.6
- net 060A6: now also RP107.7
- net 060A7: now also RP107.8
- net 060A8: now also RP106.5
- net 060A9: now also RP106.6
- net 060D0: now also RP405C.5
- net 060D1: now also RP405C.6
- net 060D10: now also RP405A.7, U217.A2
- net 060D11: now also RP405A.8, U217.A3
- net 060D12: now also RP404B.5, U217.A4
- net 060D13: now also RP404B.6, U217.A5
- net 060D14: now also RP404B.7, U217.A6
- net 060D15: now also RP404B.8, U217.A7
- net 060D16: now also RP404A.5, U215.A0, U216.A0
- net 060D17: now also RP404A.6, U215.A1, U216.A1
- net 060D18: now also RP404A.7, U215.A2, U216.A2
- net 060D19: now also RP404A.8, U215.A3, U216.A3
- net 060D2: now also RP405C.7
- net 060D20: now also RP403B.5, U215.A4, U216.A4
- net 060D21: now also RP403B.6, U215.A5, U216.A5
- net 060D22: now also RP403B.7, U215.A6, U216.A6
- net 060D23: now also RP403B.8, U215.A7, U216.A7
- net 060D24: now also RP403A.5, U214.A0
- net 060D25: now also RP403A.6, U214.A1
- net 060D26: now also RP403A.7, U214.A2
- net 060D27: now also RP403A.8, U214.A3
- net 060D28: now also RP402A.5, U214.A4
- net 060D29: now also RP402A.6, U214.A5
- net 060D3: now also RP405C.8
- net 060D30: now also RP402A.7, U214.A6
- net 060D31: now also RP402A.8, U214.A7
- net 060D4: now also RP405B.5
- net 060D5: now also RP405B.6
- net 060D6: now also RP405B.7
- net 060D7: now also RP405B.8
- net 060D8: now also RP405A.5, U217.A0
- net 060D9: now also RP405A.6, U217.A1
- net 060SIZ0: now also R108.2; no longer U102.SIZ0
- net 060SIZ1: now also R107.2; no longer U102.SIZ1
- net BCLK: now also R103.2
- net GND: now also C100A.2, C101A.2, C101B.2, C102A.2, C102B.2, C102C.2, C102D.2, C102E.2, C102F.2, C103A.2, C105A.1, C214A.1, C214A5.1, C214A6.1, C214A7.1, C214A8.1, C214A9.1, C215A.1, C216A.1, C217A.1, C501.2, CN100.GND0, CN100.GND1, CN100.GND10, CN100.GND11, CN100.GND12, CN100.GND13, CN100.GND14, CN100.GND15, CN100.GND16, CN100.GND17, CN100.GND18, CN100.GND19, CN100.GND2, CN100.GND20, CN100.GND21, CN100.GND22, CN100.GND23, CN100.GND24, CN100.GND25, CN100.GND26, CN100.GND27, CN100.GND28, CN100.GND29, CN100.GND3, CN100.GND30, CN100.GND31, CN100.GND32, CN100.GND33, CN100.GND34, CN100.GND35, CN100.GND36, CN100.GND37, CN100.GND38, CN100.GND39, CN100.GND4, CN100.GND40, CN100.GND41, CN100.GND42, CN100.GND5, CN100.GND6, CN100.GND7, CN100.GND8, CN100.GND9, R105.2, RP100A.1, RP100A.2, RP100A.3, RP100A.4, RP100B.1, RP100B.2, RP100B.3, RP100B.4, U$10.GND, U$11.GND, U$7.GND, U$8.GND, U$9.GND, U100.GND, U101.GND1, U102.DLE, U103.GND, U105.GND, U214.!LEAB, U214.GND, U215.!LEAB, U215.GND, U216.!LEAB, U216.GND, U217.!LEAB, U217.GND, VR1.GND
- net N$1: now also U102._RSTO; no longer U102.VCC0, U102.VCC1, U102.VCC10, U102.VCC11, U102.VCC12, U102.VCC13, U102.VCC14, U102.VCC15, U102.VCC16, U102.VCC17, U102.VCC18, U102.VCC19, U102.VCC2, U102.VCC20, U102.VCC21, U102.VCC22, U102.VCC23, U102.VCC24, U102.VCC25, U102.VCC26, U102.VCC27, U102.VCC28, U102.VCC29, U102.VCC3, U102.VCC30, U102.VCC31, U102.VCC32, U102.VCC33, U102.VCC34, U102.VCC35, U102.VCC36, U102.VCC37, U102.VCC38, U102.VCC39, U102.VCC4, U102.VCC40, U102.VCC5, U102.VCC6, U102.VCC7, U102.VCC8, U102.VCC9
- net PCLK: now also R100.2, U101.CP
- net PUP1: now also RP400B.5
- net _BB060: now also RP400B.6
Other:
- note added: "10nS"
- note added: "5nS"
- note added: "7407 here.."
- note added: "Delayselector"
- note added: "Populate only one"

Commit message: More stuff done.. some logic left.
Parts:
- added C200A, U201A: 100NF, A3660:C0805
- added C202A, C204: (no value), A3660:C0805
- added C203A, C206A: 100nF, A3660:C0805
- added FB200: (no value), A3660:FERRITE
- added U200: 74FCT373ASO, A3660:74FCT373ASO
- added U201: 74FCT374ASO, A3660:74FCT374ASO
- added U202: 74F32, A3660:74F32
- added U203: GAL16V8, A3660:GAL16V8
- added U204: GAL22V10, A3660:GAL22V10
- added U206: 74F139, A3660:74F139
- renumbered C214A5 to U218A, C214A6 to C219A, C214A7 to C220A, C214A8 to C221A, C214A9 to C222A, U$10 to U221, U$11 to U222, U$7 to U218, U$8 to U219, U$9 to U220
Connections:
- net N$50 renamed LEBUS7
- net N$56 renamed LEBUS6
- net N$62 renamed LEBUS5
- net N$68 renamed LEBUS4
- net N$72 renamed _DMACOE
- removed net N$47: U218.!CEBA
- removed net N$48: U218.!OEAB
- removed net N$49: U218.!OEBA
- removed net N$51: U218.!LEAB
- removed net N$52: U218.!CEAB
- removed net N$53: U219.!CEBA
- removed net N$54: U219.!OEAB
- removed net N$55: U219.!OEBA
- removed net N$57: U219.!LEAB
- removed net N$58: U219.!CEAB
- removed net N$59: U220.!CEBA
- removed net N$60: U220.!OEAB
- removed net N$61: U220.!OEBA
- removed net N$63: U220.!LEAB
- removed net N$64: U220.!CEAB
- removed net N$65: U221.!CEBA
- removed net N$66: U221.!OEAB
- removed net N$67: U221.!OEBA
- removed net N$70: U221.!CEAB
- removed net N$71: U222.!CEBA
- removed net N$73: U222.!OEBA
- removed net N$74: U222.!LEBA
- removed net N$75: U222.!LEAB
- removed net N$76: U222.!CEAB
- new net HLT: U201.D3
- new net MAS0: U204.I/O/Q7
- new net MAS1: U204.I/O/Q8
- new net MAS2: U204.I/O/Q6
- new net MAS3: U204.I/O/Q5
- new net N$22: U200.O0, U202.1B
- new net N$24: U201.O0, U203.I1
- new net N$25: U201.O1, U203.I2
- new net N$26: U201.O2, U203.I3
- new net N$27: C204.1, U204.GND
- new net N$28: C204.2, U204.VCC
- new net OEBUS4: U221.!OEAB, U221.!OEBA
- new net OEBUS5: U220.!OEAB, U220.!OEBA
- new net OEBUS6: U219.!OEAB, U219.!OEBA
- new net OEBUS7: U218.!OEAB, U218.!OEBA
- new net PUP4: RP400B.8, U222.!OEBA
- new net SLV0: U204.I/O/Q2, U206.A0B
- new net SLV1: U204.I/O/Q4, U206.A1B
- new net SLV2: U204.I/O/Q3
- new net SLV3: U204.I/O/Q1, U206.!EB
- new net _AS060: U203.I7
- new net _AVEC: U203.I8
- new net _BERR: U201.D4, U203.O3
- new net _BGACK: U200.D1, U202.2A
- new net _BGACK060: U204.I0
- new net _BR: U200.D0, U202.1A
- new net _CIIN: U200.D3, U201.D5
- new net _CPURST: U201.D7
- new net _CYCPEND: U204.I9
- new net _DSACK0: U201.D2, U203.O2
- new net _DSACK1: U201.D1, U203.OE
- new net _ETERM: U203.O6, U204.I5
- new net _LSTERM: U204.I/O/Q0
- new net _PLSTERM: FB200.2, U201.D0, U203.CLK
- new net _RAVEC: U201.O6, U203.I4
- new net _RBERR: U201.O4, U203.I5, U204.I8
- new net _RCIIN: U200.O3
- new net _RDSACK0: U203.O4, U204.I7
- new net _RDSACK1: U203.O1, U204.I6
- new net _RTERM: U203.O7
- new net _S2W: U206.!Q3B
- new net _SBGACK030: U202.2Y
- new net _SBR030: U202.1Y
- new net _SIG_LE: U206.!Q0B
- new net _STERM: FB200.1, U200.D2
- new net _TEND: U203.I6
- net +5V: now also C200A.1, C202A.1, C203A.1, C206A.1, U200.VCC, U201.VCC, U201A.1, U202.VCC1, U203.VCC, U206.VCC
- net 060D0: now also U218.A0, U219.A0, U220.A0, U221.A0
- net 060D1: now also U218.A1, U219.A1, U220.A1, U221.A1
- net 060D16: now also U222.A0
- net 060D17: now also U222.A1
- net 060D18: now also U222.A2
- net 060D19: now also U222.A3
- net 060D2: now also U218.A2, U219.A2, U220.A2, U221.A2
- net 060D20: now also U222.A4
- net 060D21: now also U222.A5
- net 060D22: now also U222.A6
- net 060D23: now also U222.A7
- net 060D3: now also U218.A3, U219.A3, U220.A3, U221.A3
- net 060D4: now also U218.A4, U219.A4, U220.A4, U221.A4
- net 060D5: now also U218.A5, U219.A5, U220.A5, U221.A5
- net 060D6: now also U218.A6, U219.A6, U220.A6, U221.A6
- net 060D7: now also U218.A7, U219.A7, U220.A7, U221.A7
- net 060SIZ0: now also U204.I3, U206.A0A
- net 060SIZ1: now also U204.I4, U206.A1A
- net A0: now also U204.I1
- net A1: now also U204.I2
- net BCLK: now also U200.EN/CLK, U201.EN/CLK, U204.I/CLK
- net D0: now also U218.B0, U222.B0
- net D1: now also U218.B1, U222.B1
- net D16: now also U219.B0
- net D17: now also U219.B1
- net D18: now also U219.B2
- net D19: now also U219.B3
- net D2: now also U218.B2, U222.B2
- net D20: now also U219.B4
- net D21: now also U219.B5
- net D22: now also U219.B6
- net D23: now also U219.B7
- net D24: now also U220.B0, U221.B0
- net D25: now also U220.B1, U221.B1
- net D26: now also U220.B2, U221.B2
- net D27: now also U220.B3, U221.B3
- net D28: now also U220.B4, U221.B4
- net D29: now also U220.B5, U221.B5
- net D3: now also U218.B3, U222.B3
- net D30: now also U220.B6, U221.B6
- net D31: now also U220.B7, U221.B7
- net D4: now also U218.B4, U222.B4
- net D5: now also U218.B5, U222.B5
- net D6: now also U218.B6, U222.B6
- net D7: now also U218.B7, U222.B7
- net GND: now also C200A.2, C202A.2, C203A.2, C206A.2, U200.!OE, U200.D4, U200.D5, U200.D6, U200.D7, U200.GND, U201.!OE, U201.GND, U201A.2, U202.GND1, U203.GND, U206.!EA, U206.GND, U218.!LEAB, U219.!LEAB, U220.!LEAB, U222.!LEAB, U222.!LEBA
- net N$23: now also U200.O1, U202.2B; no longer RP400B.8
- net R_W060: now also U218.!CEAB, U219.!CEAB, U220.!CEAB, U221.!CEAB, U222.!CEAB
- net _060RSTI: now also U201.O7, U204.I10
- net _R_W060: now also U218.!CEBA, U219.!CEBA, U220.!CEBA, U221.!CEBA, U222.!CEBA
- net _TS: now also U204.I/O/Q9

Commit message: Most stuff is there.  A lot of tidyup needed..
Parts:
- added C207, C208, C209, C211, C212, C213, C400, C402A: 100nF, A3660:C0805
- added U207, U209, U211, U213, U400: GAL22V10, A3660:GAL22V10
- added U208: GAL16V8, A3660:GAL16V8
- added U212: 74F257, A3660:74F257
- added U402: 74FCT244A, A3660:74FCT244A
- C204: value (none) -> 100nF
Connections:
- removed net N$5: C100A.1, U100.VCC
- new net 030A0: CN100.A0, U213.I/O/Q7
- new net 030A1: CN100.A1, U212.ZC
- new net 030A2: CN100.A2, U212.ZB
- new net 030A3: CN100.A3, U212.ZA
- new net FC0: U213.I/O/Q1
- new net FC1: U213.I/O/Q2
- new net FC2: U213.I/O/Q3
- new net MA24: CN100.A24, U400.I/O/Q6
- new net MA25: CN100.A25, U400.I/O/Q7
- new net MA26: CN100.A26, U400.I/O/Q8
- new net N$29: C207.1
- new net N$30: C207.2
- new net N$31: C213.1
- new net N$32: C213.2
- new net N$33: U212.I1C, U213.I/O/Q8
- new net N$34: C209.1
- new net N$35: C209.2
- new net N$36: C211.1
- new net N$37: C211.2
- new net N$38: C400.1
- new net N$39: C400.2
- new net R_W: U402.OA0
- new net SIZ0: U213.I/O/Q4
- new net SIZ1: U213.I/O/Q5
- new net _060IPEND: U402.DA3
- new net _AS: U402.OB3
- new net _BG: U209.I/O/Q4
- new net _CIOUT: U402.OA2
- new net _DS: CN100._DS, U402.OB2
- new net _DS060: U402.DB2
- new net _IACK: U212.S, U213.I/O/Q6
- new net _IPL0: U211.I10
- new net _IPL1: U211.I9
- new net _IPL2: U211.I8
- new net _PWRST: U400.I/O/Q4
- new net _RMC: U402.OA1
- new net _START: U211.I/O/Q5
- net +5V: now also C100A.1, C208.1, C212.1, C402A.2, U100.VCC, U208.VCC, U212.VCC, U402.VCC
- net 060SIZ0: now also U213.I1
- net 060SIZ1: now also U213.I2
- net A0: now also U213.I/CLK; no longer CN100.A0
- net A1: now also U213.I0; no longer CN100.A1
- net A19: now also U400.I/O/Q1
- net A2: now also U212.I1B; no longer CN100.A2
- net A20: now also U400.I/O/Q0
- net A21: now also U400.I10
- net A22: now also U400.I9
- net A23: now also U400.I8
- net A24: now also U400.I7; no longer CN100.A24
- net A25: now also U400.I6; no longer CN100.A25
- net A26: now also U400.I5; no longer CN100.A26
- net A27: now also U400.I4
- net A28: now also U400.I3
- net A29: now also U400.I2
- net A3: now also U212.I1A; no longer CN100.A3
- net A30: now also U400.I1
- net A31: now also U400.I0
- net BCLK: now also U207.I/CLK, U208.CLK, U209.I/CLK, U211.I/CLK, U400.I/CLK
- net GND: now also C208.2, C212.2, C402A.1, U208.GND, U208.OE, U212.GND, U212.I0D, U212.I1D, U402.DB0, U402.DB1, U402.GND
- net LEBUS0: now also U208.O8
- net LEBUS1: now also U208.O7
- net LEBUS2: now also U208.O6
- net LEBUS3: now also U208.O5
- net LEBUS4: now also U208.O4
- net LEBUS5: now also U208.O3
- net LEBUS6: now also U208.O2
- net LEBUS7: now also U208.O1
- net MAS0: now also U207.I0, U208.I3, U213.I/O/Q0
- net MAS1: now also U207.I1, U208.I4, U213.I10
- net MAS2: now also U207.I2, U208.I5, U213.I9
- net MAS3: now also U207.I3, U208.I6, U213.I8
- net OEBUS0: now also U207.I/O/Q8
- net OEBUS1: now also U207.I/O/Q7
- net OEBUS2: now also U207.I/O/Q6
- net OEBUS3: now also U207.I/O/Q5
- net OEBUS4: now also U207.I/O/Q4
- net OEBUS5: now also U207.I/O/Q3
- net OEBUS6: now also U207.I/O/Q2
- net OEBUS7: now also U207.I/O/Q1
- net R_W060: now also U207.I6, U400.I/O/Q3, U402.DA0
- net SLV3: now also U207.I5
- net TM0: now also U212.I0C, U213.I7
- net TM1: now also U212.I0B, U213.I6
- net TM2: now also U212.I0A, U213.I5
- net TT0: now also U213.I3
- net TT1: now also U213.I4
- net _060CIOUT: now also U402.DA2
- net _060IPL0: now also U211.I/O/Q2
- net _060IPL1: now also U211.I/O/Q1
- net _060IPL2: now also U211.I/O/Q0
- net _060RSTI: now also U209.I7, U211.I7
- net _AS060: now also U211.I0, U402.DB3
- net _AVEC060: now also U211.I/O/Q7
- net _BB060: now also U209.I2
- net _BG060: now also U209.I/O/Q5
- net _BGACK060: now also U209.I/O/Q3, U211.I5, U212.!OE, U213.I/O/Q9, U400.I/O/Q9, U402.!OEA, U402.!OEB
- net _BR060: now also U209.I3
- net _CYCPEND: now also U211.I/O/Q4
- net _DMACOE: now also U207.I/O/Q9
- net _LOCK: now also U209.I4, U402.DA1
- net _LOCKE: now also U209.I5
- net _RAVEC: now also U211.I4
- net _RBERR: now also U207.I7
- net _RCIIN: now also U211.I1
- net _RDSACK0: now also U207.I8
- net _RDSACK1: now also U207.I9
- net _S2W: now also U207.I4
- net _SBGACK030: now also U209.I0
- net _SBR030: now also U209.I1
- net _SIG_LE: now also U208.I2
- net _TA: now also U211.I2
- net _TCI: now also U211.I/O/Q6
- net _TEA: now also U211.I3
- net _TEND: now also U211.I/O/Q3
- net _TS: now also U211.I6

Commit message: A3640 schematics complete
Parts:
- added C104A, C205, C400A, C401A: 100nF, A3660:C0805
- added J100: 1X3PIN, A3660:1X3PIN
- added R400, R401: 100, A3660:R0805
- added R402, R403, R404: 470, A3660:R0805
- added RP401A, RP401B: 22, A3660:RP743-8
- added RP402B: 1K, A3660:RP743-8
- added U104: 7407, A3660:7407
- added U205: GAL22V10, A3660:GAL22V10
- added U401: GAL16V8, A3660:GAL16V8
- C202A: value (none) -> 100nF
- FB100, FB200: value (none) -> 80 Ohm / 500mA
- RP400A: value (none) -> 22
- RP400B: value (none) -> 1K
Connections:
- removed net CLKEN: U102.CLKEN
- removed net HLT: U201.D3
- removed net N$15: C103A.1, U103.VCC
- removed net N$17: R101B.1
- removed net N$19: RP400A.3
- removed net N$20: RP400A.2
- removed net N$21: RP400A.1
- removed net N$69: U221.!LEAB
- removed net N$7: RP400A.4
- removed net _IPEND060: U102._IPEND
- removed net _START: U211.I/O/Q5
- new net J100: J100.2, U400.I/O/Q2
- new net N$43: C205.1, U205.GND
- new net N$44: C205.2, U205.VCC
- new net _EMUL: CN100._EMUL, U401.I4
- new net _HLT: CN100._HLT, U201.D3
- new net _RESET: CN100._RESET, U104.3!Y
- new net _RSTO: U102._RSTO, U104.3A
- net +5V: now also C103A.1, C104A.1, C401A.1, R400.1, R402.2, R403.2, R404.2, RP400A.1, RP400A.2, RP400A.3, RP400A.4, RP401A.1, RP401A.2, RP401A.3, RP401A.4, RP401B.1, RP401B.2, RP401B.3, RP401B.4, RP402B.1, RP402B.2, RP402B.3, RP402B.4, U100.+5V, U101.+5V, U103.VCC, U104.+5V, U105.+5V, U206.+5V, U212.+5V, U401.VCC; no longer U100.VCC, U101.VCC, U105.VCC, U206.VCC, U212.VCC
- net 060D0: no longer U221.A0
- net 060D1: no longer U221.A1
- net 060D10: now also U221.A2
- net 060D11: now also U221.A3
- net 060D12: now also U221.A4
- net 060D13: now also U221.A5
- net 060D14: now also U221.A6
- net 060D15: now also U221.A7
- net 060D2: no longer U221.A2
- net 060D3: no longer U221.A3
- net 060D4: no longer U221.A4
- net 060D5: no longer U221.A5
- net 060D6: no longer U221.A6
- net 060D7: no longer U221.A7
- net 060D8: now also U221.A0
- net 060D9: now also U221.A1
- net 060SIZ0: now also RP401A.5, U205.I10
- net 060SIZ1: now also RP401A.6, U205.I6
- net BCLK: now also U205.I/CLK, U401.CLK
- net CLK90: now also R101B.1
- net D10: now also U221.B2
- net D11: now also U221.B3
- net D12: now also U221.B4
- net D13: now also U221.B5
- net D14: now also U221.B6
- net D15: now also U221.B7
- net D24: no longer U221.B0
- net D25: no longer U221.B1
- net D26: no longer U221.B2
- net D27: no longer U221.B3
- net D28: no longer U221.B4
- net D29: no longer U221.B5
- net D30: no longer U221.B6
- net D31: no longer U221.B7
- net D8: now also U221.B0
- net D9: now also U221.B1
- net FC0: now also CN100.FC0
- net FC1: now also CN100.FC1
- net FC2: now also CN100.FC2
- net GND: now also C104A.2, C400.1, C401A.2, R401.1, U101.GND, U104.GND, U221.!LEAB, U401.GND, U401.OE
- net N$1: now also C400.2, R400.2, U401.I3; no longer U102._RSTO
- net N$16: now also CN100._BOSS, R401.2; no longer U101.GND
- net N$18: now also U201.D6, U203.O8; no longer U102.R_W, U105.2A
- net N$29: now also U207.GND
- net N$30: now also U207.VCC
- net N$31: now also U213.GND
- net N$32: now also U213.VCC
- net N$34: now also U209.GND
- net N$35: now also U209.VCC
- net N$36: now also U211.GND
- net N$37: now also U211.VCC
- net N$38: now also C400A.1, U400.GND; no longer C400.1
- net N$39: now also C400A.2, U400.VCC; no longer C400.2
- net R_W: now also CN100.R_W
- net R_W060: now also RP401B.5, U102.R_W, U105.2A, U205.I0
- net SIZ0: now also CN100.SIZ0
- net SIZ1: now also CN100.SIZ1
- net SLV0: now also U205.I1
- net SLV1: now also U205.I2
- net SLV2: now also U205.I3
- net SLV3: now also U205.I4
- net TM0: now also RP401B.6
- net TM1: now also RP401B.7
- net TM2: now also RP401B.8
- net TT0: now also RP401A.7
- net TT1: now also RP401A.8
- net _060CIOUT: now also RP402B.6
- net _060EMUL: now also J100.3, U401.O8
- net _060IPEND: now also U102._IPEND
- net _060RSTI: now also U205.I/O/Q7, U401.I8
- net _AS: now also CN100._AS
- net _AS060: now also U205.I/O/Q3, U401.I1
- net _AVEC: now also CN100._AVEC
- net _BERR: now also CN100._BERR
- net _BG: now also CN100._BG, U209.I/O/Q6; no longer U209.I/O/Q4
- net _BGACK: now also CN100._BGACK
- net _BGACK060: now also U205.I/O/Q9, U209.I/O/Q7; no longer U209.I/O/Q3
- net _BR: now also CN100._BR, R403.1
- net _CIIN: now also CN100._CIIN
- net _CIOUT: now also CN100._CIOUT
- net _CPURST: now also CN100._CPURST
- net _CYCPEND: now also U205.I5
- net _DS060: now also U205.I/O/Q2
- net _DSACK0: now also CN100._DSACK0, R404.1
- net _DSACK1: now also CN100._DSACK1, R402.1
- net _IPL0: now also CN100.IPL0
- net _IPL1: now also CN100.IPL1
- net _IPL2: now also CN100.IPL2
- net _LOCK: now also RP402B.8
- net _LOCKE: now also RP402B.7
- net _LSTERM: now also U208.I8, U401.O1
- net _PLSTERM: now also CN100._STERM, U205.I7, U401.I2
- net _PWRST: now also U401.O7
- net _RMC: now also CN100._RMC
- net _RTERM: now also U205.I8, U208.I7
- net _TA: now also U205.I/O/Q8
- net _TEA: now also U205.I/O/Q5
- net _TS: now also J100.1, U205.I9
Other:
- note removed: "7407 here.."

Commit message: A3660 Complete and aprox-location of components. datasignals at bottom of cpu, address at side so it is not scattered around the board.
Parts:
- added +5V, U$2: 1X2PIN, A3660:1X2PIN
- added C105, C106, C107: 22uF, A3660:SMD-ELECTROLYTE
- added C500: 10uF, A3660:C0805
- added C502: 100nF, A3660:C0805
- added JP100: 3PAD, A3660:3PAD
- added R405, R500, R501, R502, R503, R504, R505: 4.7K, A3660:R0805
- added RP1: 4.7K, A3660:RP743-8
- added U500: 74F257, A3660:74F257
- RP400A, RP401A, RP401B: value 22 -> 1K
- renumbered J100 to J400, U201A to C201A, U218A to C218A
Connections:
- net J100 renamed J400
- new net CPUSEL: JP100.2, U500.S
- new net N$19: J400.3, R405.2
- new net N$20: R503.2, U500.I0D
- new net N$21: R504.2, U500.I0C
- new net N$40: R505.2, U500.I0A
- new net THERM0: U$2.1, U102.THERM0
- new net THERM1: U$2.2, U102.THERM1
- new net _BTT: RP1.8, U102._BTT
- new net _CLA: RP1.7, U102._CLA
- new net _CLKEN: U102.CLKEN, U500.ZB
- new net _CPUIPL0: U211.I/O/Q2, U500.I1C
- new net _CPUIPL1: U211.I/O/Q1
- new net _CPUIPL2: U211.I/O/Q0, U500.I1A, U500.I1D
- new net _SNOOP: RP1.6, U102._SNOOP
- new net _TRA: RP1.5, U102._TRA
- net +3V3: now also R500.2, R501.1, R502.2, RP1.1, RP1.2, RP1.3, RP1.4
- net +5V: now also +5V.1, C105.1, C106.1, C107.1, C500.1, C502.2, JP100.3, R405.1, R503.1, R504.1, R505.1, U500.+5V
- net BCLK: now also U500.I0B, U500.I1B
- net GND: now also +5V.2, C105.2, C106.2, C107.2, C500.2, C502.1, U500.!OE, U500.GND
- net _060EMUL: no longer J400.3
- net _060IPL0: now also R500.1, U500.ZC; no longer U211.I/O/Q2
- net _060IPL1: now also R501.2, U500.ZD; no longer U211.I/O/Q1
- net _060IPL2: now also R502.1, U500.ZA; no longer U211.I/O/Q0
- net _060RSTI: now also JP100.1
Other:
- note added: "040"
- note added: "060"
