File: A3660/A3660.brd (EAGLE design)
At the start: 207 x 98 mm, 2 parts, among them CN100 KEL8817-200-170S-F, U102 MC68040/68060

Commit message: Added and changed some in library. Added schematics for CPU, Cpuclockdriver and some of the latches
Parts:
- added C100A: 10nF, A3660:R0805
- added C101A, C103A, C105A: 100nF, A3660:R0805
- added C101B: 330nF, A3660:R0805
- added C102A, C102D: 220nF, A3660:R0805
- added C102B, C102E: 22uF, A3660:SMD-ELECTROLYTE
- added C102C, C102F: 220pF, A3660:R0805
- added C501: 10uF, A3660:R0805
- added FB100: (no value), A3660:FERRITE
- added R100, R103: 1, A3660:R0805
- added R101A, R101B, R102: 22, A3660:R0805
- added R104, R105: 4.7K, A3660:R0805
- added R107, R108: 33, A3660:R0805
- added RP100A, RP100B, RP402A, RP403A, RP403B, RP404A, RP404B, RP405A, RP405B, RP405C: 1K, A3660:RP743-8
- added RP101, RP102, RP103, RP104, RP105, RP106, RP107, RP108: 22, A3660:RP743-8
- added RP400A, RP400B: (no value), A3660:RP743-8
- added U$1: 2X22-2MM, adafruit:2X22
- added U$2: 74FCT543A, A3660:74FCT543A
- added U100: OSCILLATOR, A3660:OSCILLATOR
- added U101: 74F1803, A3660:74F1803
- added U103: DELAYLINE, A3660:DELAYLINE
- added U105: 74F04, A3660:74F04
- added VR1: LT1084-3.3, A3660:LT1084-3.3
- moved U102 5.77 mm to (173.8, 71.6)
Connections:
- new net +3V3: C102A.1, C102B.+, C102C.1, C102D.1, C102E.+, C102F.1, C501.1, U102.VCC0, U102.VCC1, U102.VCC10, U102.VCC11, U102.VCC12, U102.VCC13, U102.VCC14, U102.VCC15, U102.VCC16, U102.VCC17, U102.VCC18, U102.VCC19, U102.VCC2, U102.VCC20, U102.VCC21, U102.VCC22, U102.VCC23, U102.VCC24, U102.VCC25, U102.VCC26, U102.VCC27, U102.VCC28, U102.VCC29, U102.VCC3, U102.VCC30, U102.VCC31, U102.VCC32, U102.VCC33, U102.VCC34, U102.VCC35, U102.VCC36, U102.VCC37, U102.VCC38, U102.VCC39, U102.VCC4, U102.VCC40, U102.VCC5, U102.VCC6, U102.VCC7, U102.VCC8, U102.VCC9, VR1.OUT, VR1.OUT2
- new net +5V: C101A.1, C101B.1, C105A.2, CN100.+5V-0, CN100.+5V-1, CN100.+5V-10, CN100.+5V-11, CN100.+5V-12, CN100.+5V-13, CN100.+5V-14, CN100.+5V-15, CN100.+5V-16, CN100.+5V-17, CN100.+5V-18, CN100.+5V-19, CN100.+5V-2, CN100.+5V-20, CN100.+5V-21, CN100.+5V-22, CN100.+5V-23, CN100.+5V-3, CN100.+5V-4, CN100.+5V-5, CN100.+5V-6, CN100.+5V-7, CN100.+5V-8, CN100.+5V-9, R104.1, RP400B.1, RP400B.2, RP400B.3, RP400B.4, RP402A.1, RP402A.2, RP402A.3, RP402A.4, RP403A.1, RP403A.2, RP403A.3, RP403A.4, RP403B.1, RP403B.2, RP403B.3, RP403B.4, RP404A.1, RP404A.2, RP404A.3, RP404A.4, RP404B.1, RP404B.2, RP404B.3, RP404B.4, RP405A.1, RP405A.2, RP405A.3, RP405A.4, RP405B.1, RP405B.2, RP405B.3, RP405B.4, RP405C.1, RP405C.2, RP405C.3, RP405C.4, U101.14, U105.14, VR1.IN
- new net 10NS: R101A.2, U103.P$4
- new net 3!Y: U105.6
- new net 3A: U105.5
- new net 5NS: R101B.2, U103.P$12
- new net A0: RP108.4, RP400A.5
- new net A1: RP108.3, RP400A.6
- new net A10: RP106.2
- new net A11: RP106.1
- new net A12: RP105.4
- new net A13: RP105.3
- new net A14: RP105.2
- new net A15: RP105.1
- new net A16: RP104.4
- new net A17: RP104.3
- new net A18: RP104.2
- new net A19: RP104.1
- new net A2: RP108.2, RP400A.7
- new net A20: RP103.4
- new net A21: RP103.3
- new net A22: RP103.2
- new net A23: RP103.1
- new net A24: RP102.4
- new net A25: RP102.3
- new net A26: RP102.2
- new net A27: RP102.1
- new net A28: RP101.4
- new net A29: RP101.3
- new net A3: RP108.1, RP400A.8
- new net A30: RP101.2
- new net A31: RP101.1
- new net A4: RP107.4
- new net A5: RP107.3
- new net A6: RP107.2
- new net A7: RP107.1
- new net A8: RP106.4
- new net A9: RP106.3
- new net CLK90: CN100.EXT90, R101A.1
- new net CPUCLK: CN100.EXTCPU, R102.2
- new net N$10: RP100B.8
- new net N$11: U101.10, U101.11, U105.2
- new net N$12: R103.1, U101.3, U101.4, U101.5, U101.6, U105.1
- new net N$13: R102.1, U101.9
- new net N$14: U101.12, U103.P$1
- new net N$15: C103A.1, U103.P$14
- new net N$16: U101.1
- new net N$17: R101B.1
- new net N$18: U102.R_W, U105.3
- new net N$19: RP400A.3
- new net N$2: R107.1, U102.SIZ1
- new net N$20: RP400A.2
- new net N$21: RP400A.1
- new net N$23: RP400B.8
- new net N$3: R108.1, U102.SIZ0
- new net N$4: FB100.1, U102._TS
- new net N$5: C100A.1, U100.14
- new net N$6: R100.1, U100.8
- new net N$7: RP400A.4
- new net N$8: RP100B.6
- new net N$9: RP100B.7
- new net R_W060: RP400B.7
- new net TCK: RP100B.5, U102.TCK
- new net TDI: RP100A.7, U102.TDI
- new net TMS: RP100A.8, U102.TMS
- new net _060EMUL: R105.1, U102._CDIS, U102._MDIS
- new net _R_W060: U105.4
- new net _TBI: RP100A.5, U102._TBI
- new net _TRST: RP100A.6, U102._TRST
- new net _TS: FB100.2, R104.2
- net 060A0: now also RP108.5
- net 060A1: now also RP108.6
- net 060A10: now also RP106.7
- net 060A11: now also RP106.8
- net 060A12: now also RP105.5
- net 060A13: now also RP105.6
- net 060A14: now also RP105.7
- net 060A15: now also RP105.8
- net 060A16: now also RP104.5
- net 060A17: now also RP104.6
- net 060A18: now also RP104.7
- net 060A19: now also RP104.8
- net 060A2: now also RP108.7
- net 060A20: now also RP103.5
- net 060A21: now also RP103.6
- net 060A22: now also RP103.7
- net 060A23: now also RP103.8
- net 060A24: now also RP102.5
- net 060A25: now also RP102.6
- net 060A26: now also RP102.7
- net 060A27: now also RP102.8
- net 060A28: now also RP101.5
- net 060A29: now also RP101.6
- net 060A3: now also RP108.8
- net 060A30: now also RP101.7
- net 060A31: now also RP101.8
- net 060A4: now also RP107.5
- net 060A5: now also RP107.6
- net 060A6: now also RP107.7
- net 060A7: now also RP107.8
- net 060A8: now also RP106.5
- net 060A9: now also RP106.6
- net 060D0: now also RP405C.5
- net 060D1: now also RP405C.6
- net 060D10: now also RP405A.7
- net 060D11: now also RP405A.8
- net 060D12: now also RP404B.5
- net 060D13: now also RP404B.6
- net 060D14: now also RP404B.7
- net 060D15: now also RP404B.8
- net 060D16: now also RP404A.5
- net 060D17: now also RP404A.6
- net 060D18: now also RP404A.7
- net 060D19: now also RP404A.8
- net 060D2: now also RP405C.7
- net 060D20: now also RP403B.5
- net 060D21: now also RP403B.6
- net 060D22: now also RP403B.7
- net 060D23: now also RP403B.8
- net 060D24: now also RP403A.5, U$2.3
- net 060D25: now also RP403A.6, U$2.4
- net 060D26: now also RP403A.7, U$2.5
- net 060D27: now also RP403A.8, U$2.6
- net 060D28: now also RP402A.5, U$2.7
- net 060D29: now also RP402A.6, U$2.8
- net 060D3: now also RP405C.8
- net 060D30: now also RP402A.7, U$2.9
- net 060D31: now also RP402A.8, U$2.10
- net 060D4: now also RP405B.5
- net 060D5: now also RP405B.6
- net 060D6: now also RP405B.7
- net 060D7: now also RP405B.8
- net 060D8: now also RP405A.5
- net 060D9: now also RP405A.6
- net 060SIZ0: now also R108.2; no longer U102.SIZ0
- net 060SIZ1: now also R107.2; no longer U102.SIZ1
- net BCLK: now also R103.2
- net GND: now also C100A.2, C101A.2, C101B.2, C102A.2, C102B.-, C102C.2, C102D.2, C102E.-, C102F.2, C103A.2, C105A.1, C501.2, CN100.GND0, CN100.GND1, CN100.GND10, CN100.GND11, CN100.GND12, CN100.GND13, CN100.GND14, CN100.GND15, CN100.GND16, CN100.GND17, CN100.GND18, CN100.GND19, CN100.GND2, CN100.GND20, CN100.GND21, CN100.GND22, CN100.GND23, CN100.GND24, CN100.GND25, CN100.GND26, CN100.GND27, CN100.GND28, CN100.GND29, CN100.GND3, CN100.GND30, CN100.GND31, CN100.GND32, CN100.GND33, CN100.GND34, CN100.GND35, CN100.GND36, CN100.GND37, CN100.GND38, CN100.GND39, CN100.GND4, CN100.GND40, CN100.GND41, CN100.GND42, CN100.GND5, CN100.GND6, CN100.GND7, CN100.GND8, CN100.GND9, R105.2, RP100A.1, RP100A.2, RP100A.3, RP100A.4, RP100B.1, RP100B.2, RP100B.3, RP100B.4, U100.7, U101.7, U102.DLE, U103.P$7, U105.7, VR1.GND
- net N$1: now also U102._RSTO; no longer U102.VCC0, U102.VCC1, U102.VCC10, U102.VCC11, U102.VCC12, U102.VCC13, U102.VCC14, U102.VCC15, U102.VCC16, U102.VCC17, U102.VCC18, U102.VCC19, U102.VCC2, U102.VCC20, U102.VCC21, U102.VCC22, U102.VCC23, U102.VCC24, U102.VCC25, U102.VCC26, U102.VCC27, U102.VCC28, U102.VCC29, U102.VCC3, U102.VCC30, U102.VCC31, U102.VCC32, U102.VCC33, U102.VCC34, U102.VCC35, U102.VCC36, U102.VCC37, U102.VCC38, U102.VCC39, U102.VCC4, U102.VCC40, U102.VCC5, U102.VCC6, U102.VCC7, U102.VCC8, U102.VCC9
- net PCLK: now also R100.2, U101.8
- net PUP1: now also RP400B.5
- net _BB060: now also RP400B.6

Commit message: Most stuff is there.  A lot of tidyup needed..
Parts:
- removed U$2: 74FCT543A, A3660:74FCT543A
- added C200A, U201A: 100NF, A3660:R0805
- added C202A: (no value), A3660:R0805
- added C203A, C204, C206A, C207, C208, C209, C211, C212, C213, C400, C402A: 100nF, A3660:R0805
- added C214A, C215A, C216A, C217A, C219A, C220A, C221A, C222A, U218A: 330nF, A3660:R0805
- added FB200: (no value), A3660:FERRITE
- added U200: 74FCT373ASO, A3660:74FCT373ASO
- added U201: 74FCT374ASO, A3660:74FCT374ASO
- added U202: 74F32, A3660:74F32
- added U203, U208: GAL16V8, A3660:GAL16V8
- added U204, U207, U209, U211, U213, U400: GAL22V10, A3660:GAL22V10
- added U206: 74F139, A3660:74F139
- added U212: 74F257, A3660:74F257
- added U214, U215, U216, U217, U218, U219, U220, U221, U222: 74FCT543A, A3660:74FCT543A
- added U402: 74FCT244A, A3660:74FCT244A
- moved C102D 314.7 mm to (-87.6, 129.5), turned to 0 degrees
- moved RP404A 300.9 mm to (-119.4, 119.4), flipped to the top, turned to 0 degrees
- moved RP403A 279.7 mm to (-110.5, 119.4), flipped to the top, turned to 0 degrees
- moved RP405B 275.2 mm to (-69.8, 128.3), flipped to the top, turned to 0 degrees
- moved R104 271.3 mm to (-127.0, 142.2), flipped to the top
- moved C102C 269.7 mm to (-125.7, 129.5)
- moved RP402A 265.0 mm to (-101.6, 119.4), flipped to the top, turned to 0 degrees
- moved C102F 256.2 mm to (-40.6, 142.2), turned to 0 degrees
- moved RP404B 254.2 mm to (-61.0, 128.3), flipped to the top, turned to 0 degrees
- moved RP108 253.3 mm to (-104.1, 147.3), flipped to the top, turned to 0 degrees
- moved RP107 249.5 mm to (-95.2, 147.3), flipped to the top, turned to 0 degrees
- moved FB100 246.9 mm to (-113.0, 146.1), flipped to the top
- moved R105 246.9 mm to (-16.5, 148.6), turned to 0 degrees
- moved RP106 245.7 mm to (-86.4, 147.3), flipped to the top, turned to 0 degrees
- moved C101B 243.0 mm to (-33.0, 142.2), turned to 0 degrees
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Connections:
- removed net N$5: C100A.1, U100.14
- new net !Q1A: U206.5
- new net !Q2A: U206.6
- new net 030A0: CN100.A0, U213.25
- new net 030A1: CN100.A1, U212.12
- new net 030A2: CN100.A2, U212.7
- new net 030A3: CN100.A3, U212.4
- new net D0: CN100.D0, U218.22, U222.22
- new net D1: CN100.D1, U218.21, U222.21
- new net D10: CN100.D10
- new net D11: CN100.D11
- new net D12: CN100.D12
- new net D13: CN100.D13
- new net D14: CN100.D14
- new net D15: CN100.D15
- new net D16: CN100.D16, U216.22, U219.22
- new net D17: CN100.D17, U216.21, U219.21
- new net D18: CN100.D18, U216.20, U219.20
- new net D19: CN100.D19, U216.19, U219.19
- new net D2: CN100.D2, U218.20, U222.20
- new net D20: CN100.D20, U216.18, U219.18
- new net D21: CN100.D21, U216.17, U219.17
- new net D22: CN100.D22, U216.16, U219.16
- new net D23: CN100.D23, U216.15, U219.15
- new net D24: CN100.D24, U214.22, U215.22, U217.22, U220.22, U221.22
- new net D25: CN100.D25, U214.21, U215.21, U217.21, U220.21, U221.21
- new net D26: CN100.D26, U214.20, U215.20, U217.20, U220.20, U221.20
- new net D27: CN100.D27, U214.19, U215.19, U217.19, U220.19, U221.19
- new net D28: CN100.D28, U214.18, U215.18, U217.18, U220.18, U221.18
- new net D29: CN100.D29, U214.17, U215.17, U217.17, U220.17, U221.17
- new net D3: CN100.D3, U218.19, U222.19
- new net D30: CN100.D30, U214.16, U215.16, U217.16, U220.16, U221.16
- new net D31: CN100.D31, U214.15, U215.15, U217.15, U220.15, U221.15
- new net D4: CN100.D4, U218.18, U222.18
- new net D5: CN100.D5, U218.17, U222.17
- new net D6: CN100.D6, U218.16, U222.16
- new net D7: CN100.D7, U218.15, U222.15
- new net D8: CN100.D8
- new net D9: CN100.D9
- new net FC0: U213.18
- new net FC1: U213.19
- new net FC2: U213.20
- new net HLT: U201.8
- new net LEBUS0: U208.19, U214.1
- new net LEBUS1: U208.18, U215.1
- new net LEBUS2: U208.17, U216.1
- new net LEBUS3: U208.16, U217.1
- new net LEBUS4: U208.15, U221.1
- new net LEBUS5: U208.14, U220.1
- new net LEBUS6: U208.13, U219.1
- new net LEBUS7: U208.12, U218.1
- new net MA24: CN100.A24, U400.24
- new net MA25: CN100.A25, U400.25
- new net MA26: CN100.A26, U400.26
- new net MAS0: U204.25, U207.3, U208.4, U213.17
- new net MAS1: U204.26, U207.4, U208.5, U213.16
- new net MAS2: U204.24, U207.5, U208.6, U213.13
- new net MAS3: U204.23, U207.6, U208.7, U213.12
- new net N$22: U200.2, U202.2
- new net N$24: U201.2, U203.2
- new net N$25: U201.5, U203.3
- new net N$26: U201.6, U203.4
- new net N$27: C204.1, U204.14
- new net N$28: C204.2, U204.28
- new net N$29: C207.1
- new net N$30: C207.2
- new net N$31: C213.1
- new net N$32: C213.2
- new net N$33: U212.13, U213.26
- new net N$34: C209.1
- new net N$35: C209.2
- new net N$36: C211.1
- new net N$37: C211.2
- new net N$38: C400.1
- new net N$39: C400.2
- new net N$69: U221.14
- new net OEBUS0: U207.26, U214.13, U214.2
- new net OEBUS1: U207.25, U215.13, U215.2
- new net OEBUS2: U207.24, U216.13, U216.2
- new net OEBUS3: U207.23, U217.13, U217.2
- new net OEBUS4: U207.21, U221.13, U221.2
- new net OEBUS5: U207.20, U220.13, U220.2
- new net OEBUS6: U207.19, U219.13, U219.2
- new net OEBUS7: U207.18, U218.13, U218.2
- new net PUP4: RP400B.8, U222.2
- new net R_W: U402.18
- new net SIZ0: U213.21
- new net SIZ1: U213.23
- new net SLV0: U204.19, U206.14
- new net SLV1: U204.21, U206.13
- new net SLV2: U204.20
- new net SLV3: U204.18, U206.15, U207.9
- new net _060IPEND: U402.8
- new net _AS: U402.9
- new net _AS060: U203.8, U211.3, U402.11
- new net _AVEC: U203.9
- new net _BERR: U201.13, U203.14
- new net _BG: U209.21
- new net _BGACK: U200.4, U202.4
- new net _BGACK060: U204.3, U209.20, U211.9, U212.15, U213.27, U400.27, U402.1, U402.19
- new net _BR: U200.3, U202.1
- new net _CIIN: U200.8, U201.14
- new net _CIOUT: U402.14
- new net _CPURST: U201.18
- new net _CYCPEND: U204.13, U211.21
- new net _DMACOE: U207.27, U222.13
- new net _DS: CN100._DS, U402.7
- new net _DS060: U402.13
- new net _DSACK0: U201.7, U203.13
- new net _DSACK1: U201.4, U203.11
- new net _ETERM: U203.17, U204.9
- new net _IACK: U212.1, U213.24
- new net _IPL0: U211.16
- new net _IPL1: U211.13
- new net _IPL2: U211.12
- new net _LSTERM: U204.17
- new net _PLSTERM: FB200.2, U201.3, U203.1
- new net _PWRST: U400.21
- new net _RAVEC: U201.16, U203.5, U211.7
- new net _RBERR: U201.12, U203.6, U204.12, U207.11
- new net _RCIIN: U200.9, U211.4
- new net _RDSACK0: U203.15, U204.11, U207.12
- new net _RDSACK1: U203.12, U204.10, U207.13
- new net _RMC: U402.16
- new net _RTERM: U203.18
- new net _S2W: U206.9, U207.7
- new net _SBGACK030: U202.6, U209.3
- new net _SBR030: U202.3, U209.4
- new net _SIG_LE: U206.12, U208.3
- new net _START: U211.23
- new net _STERM: FB200.1, U200.7
- new net _TEND: U203.7, U211.20
- net +5V: now also C100A.1, C200A.1, C202A.1, C203A.1, C206A.1, C208.1, C212.1, C214A.2, C215A.2, C216A.2, C217A.2, C219A.2, C220A.2, C221A.2, C222A.2, C402A.2, U100.14, U200.20, U201.20, U201A.1, U202.14, U203.20, U206.16, U208.20, U212.16, U214.24, U215.24, U216.24, U217.24, U218.24, U218A.2, U219.24, U220.24, U221.24, U222.24, U402.20
- net 060D0: now also U218.3, U219.3, U220.3, U221.3
- net 060D1: now also U218.4, U219.4, U220.4, U221.4
- net 060D10: now also U217.5
- net 060D11: now also U217.6
- net 060D12: now also U217.7
- net 060D13: now also U217.8
- net 060D14: now also U217.9
- net 060D15: now also U217.10
- net 060D16: now also U215.3, U216.3, U222.3
- net 060D17: now also U215.4, U216.4, U222.4
- net 060D18: now also U215.5, U216.5, U222.5
- net 060D19: now also U215.6, U216.6, U222.6
- net 060D2: now also U218.5, U219.5, U220.5, U221.5
- net 060D20: now also U215.7, U216.7, U222.7
- net 060D21: now also U215.8, U216.8, U222.8
- net 060D22: now also U215.9, U216.9, U222.9
- net 060D23: now also U215.10, U216.10, U222.10
- net 060D24: now also U214.3; no longer U$2.3
- net 060D25: now also U214.4; no longer U$2.4
- net 060D26: now also U214.5; no longer U$2.5
- net 060D27: now also U214.6; no longer U$2.6
- net 060D28: now also U214.7; no longer U$2.7
- net 060D29: now also U214.8; no longer U$2.8
- net 060D3: now also U218.6, U219.6, U220.6, U221.6
- net 060D30: now also U214.9; no longer U$2.9
- net 060D31: now also U214.10; no longer U$2.10
- net 060D4: now also U218.7, U219.7, U220.7, U221.7
- net 060D5: now also U218.8, U219.8, U220.8, U221.8
- net 060D6: now also U218.9, U219.9, U220.9, U221.9
- net 060D7: now also U218.10, U219.10, U220.10, U221.10
- net 060D8: now also U217.3
- net 060D9: now also U217.4
- net 060SIZ0: now also U204.6, U206.2, U213.4
- net 060SIZ1: now also U204.7, U206.3, U213.5
- net A0: now also U204.4, U213.2
- net A1: now also U204.5, U213.3
- net A10: now also CN100.A10
- net A11: now also CN100.A11
- net A12: now also CN100.A12
- net A13: now also CN100.A13
- net A14: now also CN100.A14
- net A15: now also CN100.A15
- net A16: now also CN100.A16
- net A17: now also CN100.A17
- net A18: now also CN100.A18
- net A19: now also CN100.A19, U400.18
- net A2: now also U212.6
- net A20: now also CN100.A20, U400.17
- net A21: now also CN100.A21, U400.16
- net A22: now also CN100.A22, U400.13
- net A23: now also CN100.A23, U400.12
- net A24: now also U400.11
- net A25: now also U400.10
- net A26: now also U400.9
- net A27: now also CN100.A27, U400.7
- net A28: now also CN100.A28, U400.6
- net A29: now also CN100.A29, U400.5
- net A3: now also U212.3
- net A30: now also CN100.A30, U400.4
- net A31: now also CN100.A31, U400.3
- net A4: now also CN100.A4
- net A5: now also CN100.A5
- net A6: now also CN100.A6
- net A7: now also CN100.A7
- net A8: now also CN100.A8
- net A9: now also CN100.A9
- net BCLK: now also U200.11, U201.11, U204.2, U207.2, U208.1, U209.2, U211.2, U400.2
- net GND: now also C200A.2, C202A.2, C203A.2, C206A.2, C208.2, C212.2, C214A.1, C215A.1, C216A.1, C217A.1, C219A.1, C220A.1, C221A.1, C222A.1, C402A.1, U200.1, U200.10, U200.13, U200.14, U200.17, U200.18, U201.1, U201.10, U201A.2, U202.7, U203.10, U206.1, U206.8, U208.10, U208.11, U212.10, U212.11, U212.8, U214.12, U214.14, U215.12, U215.14, U216.12, U216.14, U217.12, U217.14, U218.12, U218.14, U218A.1, U219.12, U219.14, U220.12, U220.14, U221.12, U222.1, U222.12, U222.14, U402.10, U402.15, U402.17
- net N$23: now also U200.5, U202.5; no longer RP400B.8
- net R_W060: now also U207.10, U214.11, U215.11, U216.11, U217.11, U218.11, U219.11, U220.11, U221.11, U222.11, U400.20, U402.2
- net TM0: now also U212.14, U213.11
- net TM1: now also U212.5, U213.10
- net TM2: now also U212.2, U213.9
- net TT0: now also U213.6
- net TT1: now also U213.7
- net _060CIOUT: now also U402.6
- net _060IPL0: now also U211.19
- net _060IPL1: now also U211.18
- net _060IPL2: now also U211.17
- net _060RSTI: now also U201.19, U204.16, U209.11, U211.11
- net _AVEC060: now also U211.25
- net _BB060: now also U209.5
- net _BG060: now also U209.23
- net _BR060: now also U209.6
- net _LOCK: now also U209.7, U402.4
- net _LOCKE: now also U209.9
- net _R_W060: now also U214.23, U215.23, U216.23, U217.23, U218.23, U219.23, U220.23, U221.23, U222.23
- net _TA: now also U211.5
- net _TCI: now also U211.24
- net _TEA: now also U211.6
- net _TS: now also U204.27, U211.10

Commit message: A3640 schematics complete
Parts:
- added C104A, C205, C400A, C401A: 100nF, A3660:R0805
- added J100: 1X3PIN, A3660:1X3PIN
- added R400, R401: 100, A3660:R0805
- added R402, R403, R404: 470, A3660:R0805
- added RP401A, RP401B: 22, A3660:RP743-8
- added RP402B: 1K, A3660:RP743-8
- added U104: 7407, A3660:7407
- added U205: GAL22V10, A3660:GAL22V10
- added U401: GAL16V8, A3660:GAL16V8
- C202A: value (none) -> 100nF
- FB100, FB200: value (none) -> 80 Ohm / 500mA
- RP400A: value (none) -> 22
- RP400B: value (none) -> 1K
- moved U219 281.7 mm to (175.3, 38.1)
- moved U218 267.8 mm to (175.3, 22.9)
- moved U220 248.9 mm to (125.7, 38.1)
- moved CN100 226.8 mm to (120.0, 8.48)
- moved VR1 222.5 mm to (139.7, 83.8)
- moved U102 218.5 mm to (175.3, 72.4)
- moved U208 215.4 mm to (95.2, 68.6)
- moved U402 213.4 mm to (124.5, 53.3)
- moved U216 206.3 mm to (148.6, 38.1)
- moved U222 197.2 mm to (148.6, 22.9)
- moved U217 178.8 mm to (100.3, 22.9)
- moved U207 172.9 mm to (114.3, 68.6)
- moved U103 162.6 mm to (74.9, 31.8), turned to 90 degrees
- moved U206 160.6 mm to (69.8, 71.1)
- moved U221 160.4 mm to (125.7, 22.9)
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Connections:
- removed net !Q1A: U206.5
- removed net !Q2A: U206.6
- removed net 3!Y: U105.6
- removed net 3A: U105.5
- removed net CLKEN: U102._CLKEN
- removed net HLT: U201.8
- removed net N$15: C103A.1, U103.P$14
- removed net N$17: R101B.1
- removed net N$19: RP400A.3
- removed net N$20: RP400A.2
- removed net N$21: RP400A.1
- removed net N$69: U221.14
- removed net N$7: RP400A.4
- removed net _IPEND060: U102._IPEND
- removed net _START: U211.23
- new net J100: J100.2, U400.19
- new net N$43: C205.1, U205.14
- new net N$44: C205.2, U205.28
- new net _EMUL: CN100._EMUL, U401.5
- new net _HLT: CN100._HLT, U201.8
- new net _RESET: CN100._RESET, U104.5
- new net _RSTO: U102._RSTO, U104.6
- net +5V: now also C103A.1, C104A.1, C401A.1, R400.1, R402.2, R403.2, R404.2, RP400A.1, RP400A.2, RP400A.3, RP400A.4, RP401A.1, RP401A.2, RP401A.3, RP401A.4, RP401B.1, RP401B.2, RP401B.3, RP401B.4, RP402B.1, RP402B.2, RP402B.3, RP402B.4, U103.P$14, U104.VCC, U401.20
- net 060D0: no longer U221.3
- net 060D1: no longer U221.4
- net 060D10: now also U221.5
- net 060D11: now also U221.6
- net 060D12: now also U221.7
- net 060D13: now also U221.8
- net 060D14: now also U221.9
- net 060D15: now also U221.10
- net 060D2: no longer U221.5
- net 060D3: no longer U221.6
- net 060D4: no longer U221.7
- net 060D5: no longer U221.8
- net 060D6: no longer U221.9
- net 060D7: no longer U221.10
- net 060D8: now also U221.3
- net 060D9: now also U221.4
- net 060SIZ0: now also RP401A.5, U205.16
- net 060SIZ1: now also RP401A.6, U205.10
- net BCLK: now also U205.2, U401.1
- net CLK90: now also R101B.1
- net D10: now also U221.20
- net D11: now also U221.19
- net D12: now also U221.18
- net D13: now also U221.17
- net D14: now also U221.16
- net D15: now also U221.15
- net D24: no longer U221.22
- net D25: no longer U221.21
- net D26: no longer U221.20
- net D27: no longer U221.19
- net D28: no longer U221.18
- net D29: no longer U221.17
- net D30: no longer U221.16
- net D31: no longer U221.15
- net D8: now also U221.22
- net D9: now also U221.21
- net FC0: now also CN100.FC0
- net FC1: now also CN100.FC1
- net FC2: now also CN100.FC2
- net GND: now also C104A.2, C400.1, C401A.2, R401.1, U101.1, U104.GND, U221.14, U401.10, U401.11
- net N$1: now also C400.2, R400.2, U401.4; no longer U102._RSTO
- net N$16: now also CN100._BOSS, R401.2; no longer U101.1
- net N$18: now also U201.17, U203.19; no longer U102.R_W, U105.3
- net N$29: now also U207.14
- net N$30: now also U207.28
- net N$31: now also U213.14
- net N$32: now also U213.28
- net N$34: now also U209.14
- net N$35: now also U209.28
- net N$36: now also U211.14
- net N$37: now also U211.28
- net N$38: now also C400A.1, U400.14; no longer C400.1
- net N$39: now also C400A.2, U400.28; no longer C400.2
- net R_W: now also CN100.R_W
- net R_W060: now also RP401B.5, U102.R_W, U105.3, U205.3
- net SIZ0: now also CN100.SIZ0
- net SIZ1: now also CN100.SIZ1
- net SLV0: now also U205.4
- net SLV1: now also U205.5
- net SLV2: now also U205.6
- net SLV3: now also U205.7
- net TM0: now also RP401B.6
- net TM1: now also RP401B.7
- net TM2: now also RP401B.8
- net TT0: now also RP401A.7
- net TT1: now also RP401A.8
- net _060CIOUT: now also RP402B.6
- net _060EMUL: now also J100.3, U401.19
- net _060IPEND: now also U102._IPEND
- net _060RSTI: now also U205.25, U401.9
- net _AS: now also CN100._AS
- net _AS060: now also U205.20, U401.2
- net _AVEC: now also CN100._AVEC
- net _BERR: now also CN100._BERR
- net _BG: now also CN100._BG, U209.24; no longer U209.21
- net _BGACK: now also CN100._BGACK
- net _BGACK060: now also U205.27, U209.25; no longer U209.20
- net _BR: now also CN100._BR, R403.1
- net _CIIN: now also CN100._CIIN
- net _CIOUT: now also CN100._CIOUT
- net _CPURST: now also CN100._CPURST
- net _CYCPEND: now also U205.9
- net _DS060: now also U205.19
- net _DSACK0: now also CN100._DSACK0, R404.1
- net _DSACK1: now also CN100._DSACK1, R402.1
- net _IPL0: now also CN100._IPL0
- net _IPL1: now also CN100._IPL1
- net _IPL2: now also CN100._IPL2
- net _LOCK: now also RP402B.8
- net _LOCKE: now also RP402B.7
- net _LSTERM: now also U208.9, U401.12
- net _PLSTERM: now also CN100._PLSTERM, U205.11, U401.3
- net _PWRST: now also U401.18
- net _RMC: now also CN100._RMC
- net _RTERM: now also U205.12, U208.8
- net _TA: now also U205.26
- net _TEA: now also U205.23
- net _TS: now also J100.1, U205.13

Commit message: A3660 Complete and aprox-location of components. datasignals at bottom of cpu, address at side so it is not scattered around the board.
Parts:
- removed U201A: 100NF, A3660:R0805
- removed U218A: 330nF, A3660:R0805
- added +5V, U$2: 1X2PIN, A3660:1X2PIN
- added C105, C106, C107: 22uF, A3660:SMD-ELECTROLYTE
- added C201A: 100NF, A3660:R0805
- added C218A: 330nF, A3660:R0805
- added C500: 10uF, A3660:R0805
- added C502: 100nF, A3660:R0805
- added JP100: 3PAD, A3660:3PAD
- added R405, R500, R501, R502, R503, R504, R505: 4.7K, A3660:R0805
- added RP1: 4.7K, A3660:RP743-8
- added U500: 74F257, A3660:74F257
- RP400A, RP401A, RP401B: value 22 -> 1K
- moved C102F 332.0 mm to (201.9, 83.8)
- moved C104A 322.0 mm to (191.8, 11.4), turned to 90 degrees
- moved RP403B 308.3 mm to (180.3, 44.5), flipped to the bottom
- moved RP404B 299.7 mm to (162.6, 44.5), flipped to the bottom
- moved U104 294.0 mm to (199.4, 6.35)
- moved C402A 273.1 mm to (149.9, 58.4), turned to 90 degrees
- moved R108 271.4 mm to (148.6, 88.9), flipped to the bottom, turned to 270 degrees
- moved C222A 270.9 mm to (154.9, 21.6), turned to 90 degrees
- moved C102C 266.4 mm to (184.2, 47.0), turned to 180 degrees
- moved C219A 265.5 mm to (179.1, 36.8), turned to 90 degrees
- moved R107 264.3 mm to (148.6, 92.7), flipped to the bottom, turned to 270 degrees
- moved RP100A 252.9 mm to (124.5, 77.5), flipped to the bottom, turned to 270 degrees
- moved RP108 250.7 mm to (128.3, 62.2), flipped to the bottom, turned to 270 degrees
- moved RP402A 249.1 mm to (198.1, 44.5), flipped to the bottom
- moved RP403A 249.1 mm to (189.2, 44.5), flipped to the bottom
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- renumbered J100 to J400
Connections:
- net J100 renamed J400
- new net CPUSEL: JP100.2, U500.1
- new net N$19: J400.3, R405.2
- new net N$20: R503.2, U500.11
- new net N$21: R504.2, U500.14
- new net N$40: R505.2, U500.2
- new net THERM0: U$2.1, U102.THERM0
- new net THERM1: U$2.2, U102.THERM1
- new net _BTT: RP1.8, U102._BTT
- new net _CLA: RP1.7, U102._CLA
- new net _CLKEN: U102._CLKEN, U500.7
- new net _CPUIPL0: U211.19, U500.13
- new net _CPUIPL1: U211.18
- new net _CPUIPL2: U211.17, U500.10, U500.3
- new net _SNOOP: RP1.6, U102._SNOOP
- new net _TRA: RP1.5, U102._TRA
- net +3V3: now also R500.2, R501.1, R502.2, RP1.1, RP1.2, RP1.3, RP1.4
- net +5V: now also +5V.1, C105.+, C106.+, C107.+, C201A.1, C218A.2, C500.1, C502.2, JP100.3, R405.1, R503.1, R504.1, R505.1, U500.16; no longer U201A.1, U218A.2
- net BCLK: now also U500.5, U500.6
- net GND: now also +5V.2, C105.-, C106.-, C107.-, C201A.2, C218A.1, C500.2, C502.1, U500.15, U500.8; no longer U201A.2, U218A.1
- net _060EMUL: no longer J400.3
- net _060IPL0: now also R500.1, U500.12; no longer U211.19
- net _060IPL1: now also R501.2, U500.9; no longer U211.18
- net _060IPL2: now also R502.1, U500.4; no longer U211.17
- net _060RSTI: now also JP100.1
